File: kicad/BEMF_Controller/BEMF_Controller.kicad_sch (KiCad schematic)
At the start: 76 parts, among them J1 HEADER4VALULOK, J2 HEADER6, J3 FUSE, J4 Coil_A, J5 Coil_B, J6 Coil_C, J7 Vin, Q1 C3M0280090D, Q2 C3M0280090D, Q3 C3M0280090D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

Commit message: Changed footprint for Mosfet. Needs more work.
Parts:
- Q1, Q2, Q3, Q4, Q5, Q6: footprint Package_TO_SOT_THT:TO-247-3_Horizontal_TabDown -> main:TO-247-3_Horizontal_TabDown-with-pad; symbol Transistor_FET:C3M0280090D -> Component_Library:C3M0280090D_TO247
Connections:
- net CAP_BANK_A+: now also Q2.4 (D)
- net CAP_BANK_B+: now also Q3.4 (D)
- net CAP_BANK_C+: now also Q5.4 (D)
- net at D41.3 (K), D42.1 (A), D42.2 (A)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: now also Q4.4 (D)
- net at D11.1 (A), D11.2 (A), D9.3 (K)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: now also Q1.4 (D)
- net at D45.3 (K), D46.1 (A), D46.2 (A)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: now also Q6.4 (D)
Changed lines of the file:
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@@
 	)
 	(symbol
-		(lib_id "Transistor_FET:C3M0280090D")
+		(lib_id "Component_Library:C3M0280090D_TO247")
 		(at 195.58 180.34 0)
 		(unit 1)
@@
 			)
 		)
-		(property "Footprint" "Package_TO_SOT_THT:TO-247-3_Horizontal_TabDown"
+		(property "Footprint" "main:TO-247-3_Horizontal_TabDown-with-pad"
 			(at 200.66 182.245 0)
 			(effects
@@
 		(pin "2"
 		)
+		(pin "4"
+		)
 		(instances
 			(project ""
@@
 	)
 	(symbol
-		(lib_id "Transistor_FET:C3M0280090D")
+		(lib_id "Component_Library:C3M0280090D_TO247")
 		(at 347.98 180.34 0)
 		(unit 1)
@@
 			)
 		)
-		(property "Footprint" "Package_TO_SOT_THT:TO-247-3_Horizontal_TabDown"
+		(property "Footprint" "main:TO-247-3_Horizontal_TabDown-with-pad"
 			(at 353.06 182.245 0)
 			(effects
@@
 		(pin "2"
 		)
+		(pin "4"
+		)
 		(instances
 			(project "BEMF_Controller"
@@
 	)
 	(symbol
-		(lib_id "Transistor_FET:C3M0280090D")
+		(lib_id "Component_Library:C3M0280090D_TO247")
 		(at 271.78 144.78 0)
 		(unit 1)
@@
 			)
 		)
-		(property "Footprint" "Package_TO_SOT_THT:TO-247-3_Horizontal_TabDown"
+		(property "Footprint" "main:TO-247-3_Horizontal_TabDown-with-pad"
 			(at 276.86 146.685 0)
 			(effects
@@
 		(pin "2"
 		)
+		(pin "4"
+		)
 		(instances
 			(project "BEMF_Controller"
@@
 	)
 	(symbol
-		(lib_id "Transistor_FET:C3M0280090D")
+		(lib_id "Component_Library:C3M0280090D_TO247")
 		(at 195.58 144.78 0)
 		(unit 1)
@@
 			)
 		)
-		(property "Footprint" "Package_TO_SOT_THT:TO-247-3_Horizontal_TabDown"
+		(property "Footprint" "main:TO-247-3_Horizontal_TabDown-with-pad"
 			(at 200.66 146.685 0)
 			(effects
@@
 		(pin "2"
 		)
+		(pin "4"
+		)
 		(instances
 			(project "BEMF_Controller"
@@
 	)
 	(symbol
-		(lib_id "Transistor_FET:C3M0280090D")
+		(lib_id "Component_Library:C3M0280090D_TO247")
 		(at 271.78 180.34 0)
 		(unit 1)
@@
 			)
 		)
-		(property "Footprint" "Package_TO_SOT_THT:TO-247-3_Horizontal_TabDown"
+		(property "Footprint" "main:TO-247-3_Horizontal_TabDown-with-pad"
 			(at 276.86 182.245 0)
 			(effects
@@
 		(pin "2"
 		)
+		(pin "4"
+		)
 		(instances
 			(project "BEMF_Controller"
@@
 	)
 	(symbol
-		(lib_id "Transistor_FET:C3M0280090D")
+		(lib_id "Component_Library:C3M0280090D_TO247")
 		(at 347.98 144.78 0)
 		(unit 1)
@@
 			)
 		)
-		(property "Footprint" "Package_TO_SOT_THT:TO-247-3_Horizontal_TabDown"
+		(property "Footprint" "main:TO-247-3_Horizontal_TabDown-with-pad"
 			(at 353.06 146.685 0)
 			(effects
@@
 		(pin "2"
 		)
+		(pin "4"
+		)
 		(instances

Commit message: First version of PCB layout.
Parts:
- removed J4: Coil_A, TerminalBlock_Phoenix:TerminalBlock_Phoenix_MKDS-1,5-2-5.08_1x02_P5.08mm_Horizontal, symbol Connector:Conn_01x02_Pin
- removed J5: Coil_B, TerminalBlock_Phoenix:TerminalBlock_Phoenix_MKDS-1,5-2-5.08_1x02_P5.08mm_Horizontal, symbol Connector:Conn_01x02_Pin
- removed J6: Coil_C, TerminalBlock_Phoenix:TerminalBlock_Phoenix_MKDS-1,5-2-5.08_1x02_P5.08mm_Horizontal, symbol Connector:Conn_01x02_Pin
- added C57, C58: 1uF, Capacitor_SMD:C_1812_4532Metric, symbol Component_Library:CHV1812N250105MXT
Connections:
- net CAP_BANK_B- is gone; now on net CAP_BANK_GND: D40.3 (K), D42.3 (K), Q4.3 (S)
- net CAP_BANK_C- is gone; now on net CAP_BANK_GND: D44.3 (K), D46.3 (K), Q6.3 (S)
- net GNDD is gone; now on net GND: C44.2, C45.2, J2.1, S1.3 (2), U1.28 (GND), U8.8 (GND1), U8.9 (GND2), U9.8 (GND1), U9.9 (GND2)
- net 5V: now also C57.1, C58.1
- net GND: now also U1.13 (GND), U1.18 (GND), U1.23 (GND), U1.3 (GND), U1.8 (GND), C57.2, C58.2; no longer U5.4 (GND), U6.4 (GND), U7.4 (GND)
- net COIL_B_-: now reaches D41.3 (K), D42.1 (A), D42.2 (A), Q4.2 (D), Q4.4 (D)
- net COIL_A_-: now reaches D11.1 (A), D11.2 (A), D9.3 (K), Q1.2 (D), Q1.4 (D)
- net COIL_C_-: now reaches D45.3 (K), D46.1 (A), D46.2 (A), Q6.2 (D), Q6.4 (D)
- net CAP_BANK_A- renamed CAP_BANK_GND
- net CAP_BANK_GND: now also U5.4 (GND), U6.4 (GND), U7.4 (GND)
- net COM_A renamed COIL_A_+
- net COM_B renamed COIL_B_+
- net COM_C renamed COIL_C_+
