File: kicad/BEMF_Controller/BEMF_Controller.kicad_pcb (KiCad board)
At the start: 2 copper layers, 195 parts, among them J1 HEADER4VALULOK, J2 HEADER6, J3 FUSE, J4 Coil_A, J5 Coil_B, J6 Coil_C, J7 Vin, Q1 C3M0280090D, Q2 C3M0280090D, Q3 C3M0280090D, Q4 C3M0280090D, Q5 C3M0280090D, Q6 C3M0280090D, U1 Raspberry Pi Pico, U10 OPA2376AIDR, U11 ADC108S022CIMTX/NOPB, U12 OPA2376AIDR, U13 INA181, U14 INA181, U15 INA181, U2 INA181, U3 V_REG_78XX, U4 TC1240A, U5 DGD2304, U6 DGD2304, U7 DGD2304, U8 ISO7760FQDWRQ1, U9 ISO7760FQDWRQ1

Commit message: Some further work on pcb
Parts:
- moved D44 205.0 mm to (-217.8, 186.1)
- moved D43 205.0 mm to (-205.1, 177.7)
- moved D45 205.0 mm to (-211.4, 186.1)
- moved R31 197.0 mm to (103.5, 144.2), turned to 180 degrees
- moved U11 181.1 mm to (141.7, 165.7)
- moved U12 162.6 mm to (125.0, 165.8)
- moved J5 48.5 mm to (86.5, 126.8)
- moved D22 43.2 mm to (136.6, 129.3)
- moved D21 40.2 mm to (126.0, 130.1)
- moved D20 30.4 mm to (122.0, 145.6)
- moved D40 19.4 mm to (93.3, 138.8), turned to 90 degrees
- moved C25 19.4 mm to (119.8, 106.8)
- moved D41 12.2 mm to (81.0, 149.9), turned to 90 degrees
- moved D39 9.57 mm to (81.0, 138.8), turned to 90 degrees
- moved D42 5.53 mm to (93.0, 149.6), turned to 90 degrees
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Routing:
- added copper zone on F.Cu, net /CAP_BANK_B+

Commit message: First version of PCB layout.
Parts:
- removed J4: Coil_A, TerminalBlock_Phoenix:TerminalBlock_Phoenix_MKDS-1,5-2-5.08_1x02_P5.08mm_Horizontal
- removed J5: Coil_B, TerminalBlock_Phoenix:TerminalBlock_Phoenix_MKDS-1,5-2-5.08_1x02_P5.08mm_Horizontal
- removed J6: Coil_C, TerminalBlock_Phoenix:TerminalBlock_Phoenix_MKDS-1,5-2-5.08_1x02_P5.08mm_Horizontal
- removed U$6, U$7, U$8: PAD, main:PAD
- added ?: , , F.Cu at (113.9, 160.2)
- added ?: , , F.Cu at (113.8, 104.2)
- added ?: , , F.Cu at (124.3, 91.0)
- added ?: , , F.Cu at (124.1, 34.5)
- added ?: , , F.Cu at (123.8, 147.2)
- added ?: , , F.Cu at (113.9, 48.0)
- added C57: 1uF, Capacitor_SMD:C_1812_4532Metric, F.Cu at (142.8, 146.5)
- added C58: 1uF, Capacitor_SMD:C_1812_4532Metric, F.Cu at (174.5, 116.3)
- moved D44 346.2 mm to (127.0, 155.2), turned to 90 degrees
- moved D45 328.0 mm to (114.3, 147.8), turned to 180 degrees
- moved U$11 313.3 mm to (144.2, 173.8)
- moved D43 311.1 mm to (105.6, 161.3), turned to 180 degrees
- moved Q2 300.4 mm to (99.3, 58.9), turned to 90 degrees
- moved R18 297.3 mm to (104.8, 169.2), turned to 0 degrees
- moved Q6 288.8 mm to (99.6, 152.7), turned to 90 degrees
- moved R19 280.1 mm to (104.1, 155.2), turned to 0 degrees
- moved Q1 275.3 mm to (99.5, 40.5), turned to 90 degrees
- moved R14 270.3 mm to (104.6, 57.0), turned to 0 degrees
- moved Q5 265.5 mm to (99.7, 171.2), turned to 90 degrees
- moved R15 263.8 mm to (104.1, 43.0), turned to 0 degrees
- moved R17 260.1 mm to (104.1, 99.2), turned to 0 degrees
- moved C44 234.2 mm to (174.5, 123.7), turned to 90 degrees
- moved C46 225.8 mm to (151.1, 22.7), turned to -90 degrees
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Connections:
- net /Analog_IO/VSENSE_A renamed VSENSE_A
- net /Analog_IO/VSENSE_B renamed VSENSE_B
- net /Analog_IO/VSENSE_C renamed VSENSE_C
- net /COM_A renamed COIL_A_+
- net /COM_B renamed COIL_B_+
- net /COM_C renamed COIL_C_+
- net Net-(D41-K) renamed COIL_B_-
- net Net-(D45-K) renamed COIL_C_-
- net Net-(D47-K) renamed /Analog_IO/VSENSE_A_IN
- net Net-(D48-K) renamed /Analog_IO/VSENSE_C_IN
- net Net-(D51-K) renamed /Analog_IO/VSENSE_B_IN
- net Net-(D9-K) renamed COIL_A_-
- C10 pad +: /Cap_banks/CAP_BANK_A+ -> CAP_BANK_A+
- C18 pad 1: /V_RAW -> V_RAW
- C19 pad 1: /V_RAW -> V_RAW
- C20 pad 1: /V_RAW -> V_RAW
- C22 pad 2: /Cap_banks/SHUNT_A+ -> SHUNT_A+
- C23 pad 1: /Cap_banks/CAP_BANK_A+ -> CAP_BANK_A+
- C26 pad -: /Cap_banks/SHUNT_B+ -> SHUNT_B+
- C27 pad +: /Cap_banks/CAP_BANK_B+ -> CAP_BANK_B+
- C29 pad 2: /Cap_banks/SHUNT_B+ -> SHUNT_B+
- C30 pad 1: /Cap_banks/CAP_BANK_B+ -> CAP_BANK_B+
- C34 pad -: /Cap_banks/SHUNT_C+ -> SHUNT_C+
- C35 pad +: /Cap_banks/CAP_BANK_C+ -> CAP_BANK_C+
- C37 pad 2: /Cap_banks/SHUNT_C+ -> SHUNT_C+
- C38 pad 1: /Cap_banks/CAP_BANK_C+ -> CAP_BANK_C+
- C4 pad +: /V_RAW -> V_RAW
- C41 pad 2: GNDA -> CAP_BANK_GND
- C42 pad 2: GNDA -> CAP_BANK_GND
- C44 pad 2: GNDD -> GND
- C45 pad 2: GNDD -> GND
- C47 pad 2: GNDA -> CAP_BANK_GND
- C48 pad 2: GND -> CAP_BANK_GND
- C49 pad 2: GND -> CAP_BANK_GND
- C5 pad +: /V_RAW -> V_RAW
- C50 pad 2: GND -> CAP_BANK_GND
- C51 pad 2: GND -> CAP_BANK_GND
- C52 pad 2: GND -> CAP_BANK_GND
- C53 pad 2: GND -> CAP_BANK_GND
- C56 pad 2: GNDD -> GND
- C8 pad -: /Cap_banks/SHUNT_A+ -> SHUNT_A+
- D1 pad C: /V_RAW -> V_RAW
- D10 pad 3: /Cap_banks/SHUNT_A+ -> SHUNT_A+
- D11 pad 3: /CAP_BANK_A- -> CAP_BANK_GND
- D12 pad 3: /Cap_banks/SHUNT_A+ -> SHUNT_A+
- D16 pad 1: /Cap_banks/CAP_BANK_A+ -> CAP_BANK_A+
- D16 pad 2: /Cap_banks/CAP_BANK_A+ -> CAP_BANK_A+
- D17 pad 1: /Cap_banks/CAP_BANK_A+ -> CAP_BANK_A+
- D17 pad 2: /Cap_banks/CAP_BANK_A+ -> CAP_BANK_A+
- D18 pad 1: /Cap_banks/CAP_BANK_A+ -> CAP_BANK_A+
- D18 pad 2: /Cap_banks/CAP_BANK_A+ -> CAP_BANK_A+
- D19 pad 1: /Cap_banks/CAP_BANK_B+ -> CAP_BANK_B+
- D19 pad 2: /Cap_banks/CAP_BANK_B+ -> CAP_BANK_B+
- D19 pad 3: /Cap_banks/V_RAW -> V_RAW
- D20 pad 3: /Cap_banks/SHUNT_B+ -> SHUNT_B+
- D21 pad 3: /Cap_banks/SHUNT_B+ -> SHUNT_B+
- D22 pad 3: /Cap_banks/SHUNT_B+ -> SHUNT_B+
- D26 pad 1: /Cap_banks/CAP_BANK_B+ -> CAP_BANK_B+
- D26 pad 2: /Cap_banks/CAP_BANK_B+ -> CAP_BANK_B+
- D27 pad 1: /Cap_banks/CAP_BANK_B+ -> CAP_BANK_B+
- D27 pad 2: /Cap_banks/CAP_BANK_B+ -> CAP_BANK_B+
- D28 pad 1: /Cap_banks/CAP_BANK_B+ -> CAP_BANK_B+
- D28 pad 2: /Cap_banks/CAP_BANK_B+ -> CAP_BANK_B+
- D29 pad 1: /Cap_banks/CAP_BANK_C+ -> CAP_BANK_C+
- D29 pad 2: /Cap_banks/CAP_BANK_C+ -> CAP_BANK_C+
- D29 pad 3: /Cap_banks/V_RAW -> V_RAW
- D30 pad 3: /Cap_banks/SHUNT_C+ -> SHUNT_C+
- D31 pad 3: /Cap_banks/SHUNT_C+ -> SHUNT_C+
- D32 pad 3: /Cap_banks/SHUNT_C+ -> SHUNT_C+
- D36 pad 1: /Cap_banks/CAP_BANK_C+ -> CAP_BANK_C+
- D36 pad 2: /Cap_banks/CAP_BANK_C+ -> CAP_BANK_C+
- D37 pad 1: /Cap_banks/CAP_BANK_C+ -> CAP_BANK_C+
- D37 pad 2: /Cap_banks/CAP_BANK_C+ -> CAP_BANK_C+
- D38 pad 1: /Cap_banks/CAP_BANK_C+ -> CAP_BANK_C+
- D38 pad 2: /Cap_banks/CAP_BANK_C+ -> CAP_BANK_C+
- D39 pad 1: /CAP_BANK_B+ -> CAP_BANK_B+
- D39 pad 2: /CAP_BANK_B+ -> CAP_BANK_B+
- D40 pad 3: /CAP_BANK_B- -> CAP_BANK_GND
- D41 pad 1: /CAP_BANK_B+ -> CAP_BANK_B+
- D41 pad 2: /CAP_BANK_B+ -> CAP_BANK_B+
- D42 pad 3: /CAP_BANK_B- -> CAP_BANK_GND
- D43 pad 1: /CAP_BANK_C+ -> CAP_BANK_C+
- D43 pad 2: /CAP_BANK_C+ -> CAP_BANK_C+
- D44 pad 3: /CAP_BANK_C- -> CAP_BANK_GND
- D45 pad 1: /CAP_BANK_C+ -> CAP_BANK_C+
- D45 pad 2: /CAP_BANK_C+ -> CAP_BANK_C+
- D46 pad 3: /CAP_BANK_C- -> CAP_BANK_GND
- D5 pad 1: /CAP_BANK_A+ -> CAP_BANK_A+
- D5 pad 2: /CAP_BANK_A+ -> CAP_BANK_A+
- D50 pad 2: GNDA -> CAP_BANK_GND
- D53 pad 2: GNDA -> CAP_BANK_GND
- D59 pad 2: /Analog_IO/VSENSE_IN -> VSENSE_IN
- D6 pad 1: /Cap_banks/CAP_BANK_A+ -> CAP_BANK_A+
- D6 pad 2: /Cap_banks/CAP_BANK_A+ -> CAP_BANK_A+
- D6 pad 3: /Cap_banks/V_RAW -> V_RAW
- D60 pad 1: /Analog_IO/VSENSE_IN -> VSENSE_IN
- D60 pad 2: GNDA -> GND
- D62 pad 2: GNDA -> CAP_BANK_GND
- D7 pad 3: /CAP_BANK_A- -> CAP_BANK_GND
- D8 pad 3: /Cap_banks/SHUNT_A+ -> SHUNT_A+
- D9 pad 1: /CAP_BANK_A+ -> CAP_BANK_A+
- D9 pad 2: /CAP_BANK_A+ -> CAP_BANK_A+
- J2 pad 1: GNDD -> GND
- J3 pad 2A: /V_RAW -> V_RAW
- J3 pad 2B: /V_RAW -> V_RAW
- JP2 pad 2: /Cap_banks/CAP_BANK_A+ -> CAP_BANK_A+
- JP4 pad 2: /Cap_banks/CAP_BANK_B+ -> CAP_BANK_B+
- JP6 pad 2: /Cap_banks/CAP_BANK_C+ -> CAP_BANK_C+
- JP7 pad 1: /V_RAW -> V_RAW
- Q1 pad 3: /CAP_BANK_A- -> CAP_BANK_GND
- Q2 pad 2: /CAP_BANK_A+ -> CAP_BANK_A+
- Q2 pad 4: /CAP_BANK_A+ -> CAP_BANK_A+
- Q3 pad 2: /CAP_BANK_B+ -> CAP_BANK_B+
- Q3 pad 4: /CAP_BANK_B+ -> CAP_BANK_B+
- Q4 pad 3: /CAP_BANK_B- -> CAP_BANK_GND
- Q5 pad 2: /CAP_BANK_C+ -> CAP_BANK_C+
- Q5 pad 4: /CAP_BANK_C+ -> CAP_BANK_C+
- Q6 pad 3: /CAP_BANK_C- -> CAP_BANK_GND
- R12 pad 1: /VSENSE_IN -> VSENSE_IN
- R12 pad 2: /V_RAW -> V_RAW
- R13 pad 2: /VSENSE_IN -> VSENSE_IN
- R20 pad 2: /Analog_IO/CAP_BANK_A+ -> CAP_BANK_A+
- R21 pad 1: GNDA -> CAP_BANK_GND
- R22 pad 2: /Analog_IO/CAP_BANK_C+ -> CAP_BANK_C+
- R23 pad 1: GNDA -> CAP_BANK_GND
- R25 pad 2: /Analog_IO/CAP_BANK_B+ -> CAP_BANK_B+
- R26 pad 1: /Analog_IO/VSENSE_IN -> VSENSE_IN
- R28 pad 1: GNDA -> CAP_BANK_GND
- R30 pad 1: /Cap_banks/SHUNT_A+ -> SHUNT_A+
- R30 pad 2: /Cap_banks/CAP_BANK_A- -> CAP_BANK_GND
- R31 pad 1: /Cap_banks/SHUNT_B+ -> SHUNT_B+
- R31 pad 2: /Cap_banks/CAP_BANK_B- -> CAP_BANK_GND
- R32 pad 1: /Cap_banks/SHUNT_C+ -> SHUNT_C+
- R32 pad 2: /Cap_banks/CAP_BANK_C- -> CAP_BANK_GND
- R34 pad 1: GND -> CAP_BANK_GND
- R36 pad 1: GND -> CAP_BANK_GND
- R38 pad 1: GND -> CAP_BANK_GND
- R9 pad 2: /Current_sense/CAP_BANK_A- -> CAP_BANK_GND
- S1 pad 3: GNDD -> GND
- U1 pad 13: unconnected-(U1-GND-Pad13) -> GND
- U1 pad 18: unconnected-(U1-GND-Pad18) -> GND
- U1 pad 23: unconnected-(U1-GND-Pad23) -> GND
- U1 pad 28: GNDD -> GND
- U1 pad 3: unconnected-(U1-GND-Pad3) -> GND
- U1 pad 31: /ISENSE -> ISENSE
- U1 pad 32: /VSENSE -> VSENSE
- U1 pad 4: /SPI0_SCK -> SPI0_SCK
- U1 pad 5: /SPI0_TX -> SPI0_TX
- U1 pad 6: /SPI0_RX -> SPI0_RX
- U1 pad 7: /SPI0_CSn -> SPI0_CSn
- U1 pad 8: unconnected-(U1-GND-Pad8) -> GND
- U10 pad 1: /Analog_IO/VSENSE -> VSENSE
- U10 pad 2: /Analog_IO/VSENSE -> VSENSE
- U11 pad 1: /Analog_IO/SPI0_CSn -> SPI0_CSn
- U11 pad 10: /Analog_IO/ISENSE_B -> ISENSE_B
- U11 pad 11: /Analog_IO/ISENSE_A -> ISENSE_A
- U11 pad 12: GNDD -> GND
- U11 pad 14: /Analog_IO/SPI0_TX -> SPI0_TX
- U11 pad 15: /Analog_IO/SPI0_RX -> SPI0_RX
- U11 pad 16: /Analog_IO/SPI0_SCK -> SPI0_SCK
- U11 pad 9: /Analog_IO/ISENSE_C -> ISENSE_C
- U13 pad 1: /Current_sense/ISENSE_A -> ISENSE_A
- U13 pad 2: GND -> CAP_BANK_GND
- U13 pad 3: /Current_sense/SHUNT_A+ -> SHUNT_A+
- U13 pad 4: /Current_sense/SHUNT_A- -> CAP_BANK_GND
- U14 pad 1: /Current_sense/ISENSE_B -> ISENSE_B
- U14 pad 2: GND -> CAP_BANK_GND
- U14 pad 3: /Current_sense/SHUNT_B+ -> SHUNT_B+
- U14 pad 4: /Current_sense/SHUNT_B- -> CAP_BANK_GND
- U15 pad 1: /Current_sense/ISENSE_C -> ISENSE_C
- U15 pad 2: GND -> CAP_BANK_GND
- U15 pad 3: /Current_sense/SHUNT_C+ -> SHUNT_C+
- U15 pad 4: /Current_sense/SHUNT_C- -> CAP_BANK_GND
- U2 pad 1: /Current_sense/ISENSE -> ISENSE
- U2 pad 3: /Current_sense/CAP_BANK_A- -> CAP_BANK_GND
- U5 pad 4: GND -> CAP_BANK_GND
- U6 pad 4: GND -> CAP_BANK_GND
- U7 pad 4: GND -> CAP_BANK_GND
- U8 pad 8: GNDD -> GND
- U8 pad 9: GNDD -> GND
- U9 pad 8: GNDD -> GND
- U9 pad 9: GNDD -> GND
Routing:
- net 3.3V: track 101.1 -> 478.2 mm, vias 2 -> 12
- net ISENSE_A: track 0.00 -> 182.2 mm, vias 0 -> 8
- net ISENSE: track 0.00 -> 180.1 mm, vias 0 -> 7
- net 5V: track 138.6 -> 287.4 mm, vias 3 -> 4
- net /Analog_IO/VSENSE_C_IN: track 0.00 -> 146.0 mm, vias 0 -> 4
- net /10V: track 60.0 -> 188.0 mm, vias 4 -> 7
- net ISENSE_C: track 0.00 -> 118.3 mm, vias 0 -> 4
- net ISENSE_B: track 0.00 -> 116.7 mm, vias 0 -> 4
- net Net-(U2-REF): track 127.6 -> 19.3 mm, vias 2 -> 0
- net /Analog_IO/VSENSE_B_IN: track 0.00 -> 105.3 mm, vias 0 -> 2
- net VSENSE: track 0.00 -> 103.4 mm, vias 0 -> 2
- net SPI0_CSn: track 0.00 -> 102.3 mm, vias 0 -> 2
- net /Analog_IO/VSENSE_A_IN: track 0.00 -> 101.3 mm, vias 0 -> 2
- net GNDA: track 0.00 -> 86.8 mm, vias 0 -> 4
- net SPI0_SCK: track 0.00 -> 84.5 mm, vias 0 -> 1
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- added copper zone on B.Cu, net CAP_BANK_A+
- added copper zone on F.Cu, net CAP_BANK_A+
- added copper zone on B.Cu, net CAP_BANK_B+
- added copper zone on F.Cu, net CAP_BANK_B+
- added copper zone on B.Cu, net CAP_BANK_C+
- added copper zone on F.Cu, net CAP_BANK_C+
- added copper zone on B.Cu, net CAP_BANK_GND
- added copper zone on F.Cu, net CAP_BANK_GND
- added copper zone on F.Cu, net COIL_A_-
- added copper zone on F.Cu, net COIL_B_-
- added copper zone on F.Cu, net COIL_C_-
- added copper zone on F.Cu, net GNDA
- added copper zone on F.Cu, net Net-(D13-K)
- added copper zone on F.Cu, net Net-(D14-K)
- added copper zone on F.Cu, net Net-(D15-K)
- added copper zone on F.Cu, net Net-(D16-K)
- added copper zone on F.Cu, net Net-(D17-K)
- added copper zone on F.Cu, net Net-(D18-K)
- added copper zone on F.Cu, net Net-(D23-K)
- added copper zone on F.Cu, net Net-(D24-K)
- added copper zone on F.Cu, net Net-(D25-K)
- added copper zone on F.Cu, net Net-(D26-K)
- added copper zone on F.Cu, net Net-(D27-K)
- added copper zone on F.Cu, net Net-(D28-K)
- added copper zone on F.Cu, net Net-(D33-K)
- added copper zone on F.Cu, net Net-(D34-K)
- added copper zone on F.Cu, net Net-(D35-K)
- added copper zone on F.Cu, net Net-(D36-K)
- added copper zone on F.Cu, net Net-(D37-K)
- added copper zone on F.Cu, net Net-(D38-K)
- added copper zone on B.Cu, net SHUNT_A+
- added copper zone on F.Cu, net SHUNT_A+
- added copper zone on B.Cu, net SHUNT_B+
- added copper zone on F.Cu, net SHUNT_B+
- added copper zone on B.Cu, net SHUNT_C+
- added copper zone on F.Cu, net SHUNT_C+
- added copper zone on F.Cu, net V_RAW
- removed copper zone on F.Cu, net /CAP_BANK_B+
- removed copper zone on B.Cu, net /Current_sense/CAP_BANK_A-
- removed copper zone on F.Cu, net /Current_sense/CAP_BANK_A-
- removed copper zone on F.Cu, net /V_RAW
Other:
- board text added: "1uF"
- board text removed: "A"
- board text removed: "A HIGH"
- board text removed: "A LOW"
- board text removed: "B"
- board text removed: "B HIGH"
- board text removed: "B LOW"
- board text removed: "C"
- board text removed: "C HIGH"
- board text removed: "C LOW"
- board text removed: "Gate Drivers"
- board text removed: "SEM"

Commit message: Feature complete, zero eroors in pcb. Still lot of warnings.
Parts:
- removed ? (x6): , 
- removed U$10, U$11, U$12: SCREW, main:M3HOLE
- added C59: 22nF, Capacitor_SMD:C_0805_2012Metric, F.Cu at (305.0, 121.7)
- added C60: 1uF, Capacitor_SMD:C_1812_4532Metric, F.Cu at (293.5, 107.0)
- added C61: 1uF, Capacitor_SMD:C_1812_4532Metric, F.Cu at (115.0, 126.2)
- added C62: 1uF, Capacitor_SMD:C_1812_4532Metric, F.Cu at (271.2, 166.6)
- added C63: 1uF, Capacitor_SMD:C_1812_4532Metric, F.Cu at (292.7, 137.5)
- added C64: 1uF, Capacitor_SMD:C_1812_4532Metric, F.Cu at (262.0, 166.3)
- added C65: 1uF, Capacitor_SMD:C_1812_4532Metric, F.Cu at (131.7, 103.6)
- added C66: 1uF, Capacitor_SMD:C_1812_4532Metric, F.Cu at (131.8, 156.5)
- added C67: 1uF, Capacitor_SMD:C_1812_4532Metric, F.Cu at (132.2, 210.5)
- added C68: 1uF, Capacitor_SMD:C_1812_4532Metric, F.Cu at (134.5, 63.3)
- added C69: 470uF, main:CPOL-RADIAL-5MM-10MM, F.Cu at (114.5, 162.8)
- added C70: 470uF, main:CPOL-RADIAL-5MM-10MM, F.Cu at (114.5, 109.2)
- added D54: 1N4148WS, Diode_SMD:D_SOD-323, F.Cu at (112.9, 132.8)
- added D55: 1N4148WS, Diode_SMD:D_SOD-323, F.Cu at (285.0, 123.0)
- added D56: 1N4148WS, Diode_SMD:D_SOD-323, F.Cu at (290.0, 122.0)
- added D57: SMD-DIODE-100V-200MA(SOD-123), main:SOD-123, F.Cu at (130.1, 116.9)
- added D58: SMD-DIODE-100V-200MA(SOD-123), main:SOD-123, F.Cu at (130.5, 169.2)
- added D63: SMD-DIODE-100V-200MA(SOD-123), main:SOD-123, F.Cu at (130.2, 222.8)
- added D64: FSV20150V, Package_TO_SOT_SMD:TO-277A, F.Cu at (136.8, 57.0)
- added J4: HEADER6, main:6PINVALULOK, F.Cu at (302.7, 129.6)
- added J5: Load, TerminalBlock_Phoenix:TerminalBlock_Phoenix_MKDS-1,5-2-5.08_1x02_P5.08mm_Horizontal, F.Cu at (127.1, 60.1)
- added JP10: SolderJumper_3_Bridged12, Jumper:SolderJumper-3_P1.3mm_Bridged2Bar12_RoundedPad1.0x1.5mm, F.Cu at (307.2, 141.4)
- added JP8: SolderJumper_3_Bridged12, Jumper:SolderJumper-3_P1.3mm_Bridged2Bar12_RoundedPad1.0x1.5mm, F.Cu at (298.5, 141.3)
- added JP9: SolderJumper_3_Bridged12, Jumper:SolderJumper-3_P1.3mm_Bridged2Bar12_RoundedPad1.0x1.5mm, F.Cu at (303.2, 141.4)
- added Q11: C3M0280090D, Package_TO_SOT_THT:TO-247-3_Horizontal_TabDown, F.Cu at (123.3, 201.4)
- added Q7: C3M0280090D, Package_TO_SOT_THT:TO-247-3_Horizontal_TabDown, F.Cu at (123.0, 96.2)
- added Q9: C3M0280090D, Package_TO_SOT_THT:TO-247-3_Horizontal_TabDown, F.Cu at (123.0, 148.6)
- added R39: 47k, main:1206, F.Cu at (299.0, 121.7)
- added R40: 47k, main:1206, F.Cu at (302.0, 121.7)
- added R41: 192k, main:1206, F.Cu at (112.9, 138.6)
- added R42: 2.2k, main:1206, F.Cu at (115.5, 120.8)
- added R43: 1k, main:1206, F.Cu at (292.2, 121.2)
- added R44: 10, Resistor_THT:R_Axial_DIN0411_L9.9mm_D3.6mm_P15.24mm_Horizontal, F.Cu at (124.0, 101.9)
- added R46: 10, Resistor_THT:R_Axial_DIN0411_L9.9mm_D3.6mm_P15.24mm_Horizontal, F.Cu at (124.0, 154.2)
- added R48: 10, Resistor_THT:R_Axial_DIN0411_L9.9mm_D3.6mm_P15.24mm_Horizontal, F.Cu at (123.0, 207.5)
- added U16: OPA2376AIDR, footprints:D8, F.Cu at (291.6, 129.0)
- added U18: ISO7760FQDWRQ1, Package_SO:SOIC-16W_7.5x10.3mm_P1.27mm, F.Cu at (266.4, 157.7)
- added U19: DGD2304, main:SOIC8, F.Cu at (131.2, 111.9)
- added U20: DGD2304, main:SOIC8, F.Cu at (131.6, 164.4)
- added U21: DGD2304, main:SOIC8, F.Cu at (131.3, 217.4)
- Q1, Q2, Q3, Q4, Q5, Q6: footprint main:TO-247-3_Horizontal_TabDown-with-pad -> Package_TO_SOT_THT:TO-247-3_Horizontal_TabDown
- R20, R22, R25: value 180k -> 192k
- moved S1 128.5 mm to (302.7, 148.2)
- moved C47 128.4 mm to (196.4, 169.8)
- moved R1 128.4 mm to (296.2, 155.2)
- moved R2 128.3 mm to (293.5, 155.2)
- moved R3 128.3 mm to (290.8, 155.2)
- moved R4 128.3 mm to (296.2, 149.9)
- moved R5 128.3 mm to (293.5, 149.9)
- moved R6 128.3 mm to (290.8, 149.9)
- moved C17 128.3 mm to (261.1, 64.7)
- moved C43 128.3 mm to (271.1, 126.2)
- moved C46 128.3 mm to (271.4, 67.5)
- moved D59 128.3 mm to (266.2, 110.8)
- moved J1 128.3 mm to (304.6, 110.6)
- moved R10 128.3 mm to (266.6, 64.0)
- moved R11 128.3 mm to (266.6, 69.5)
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Connections:
- net /HALL_A renamed HALL_A
- net /HALL_B renamed HALL_B
- net /HALL_C renamed HALL_C
- C9 pad 1: /THROTTLE -> THROTTLE
- J1 pad 1: unconnected-(J1-Pad1) -> Net-(J1-Pad1)
- R7 pad 2: /THROTTLE -> THROTTLE
- R8 pad 2: /THROTTLE -> THROTTLE
- U1 pad 14: unconnected-(U1-GPIO10-Pad14) -> /DA_O
- U1 pad 15: unconnected-(U1-GPIO11-Pad15) -> /DB_O
- U1 pad 16: unconnected-(U1-GPIO12-Pad16) -> /DC_O
- U1 pad 31: ISENSE -> ISENSE_A_HALL_1
- U1 pad 32: VSENSE -> ISENSE_B_HALL_2
- U1 pad 34: /THROTTLE -> ISENSE_C_HALL_3
- U11 pad 10: ISENSE_B -> THROTTLE
- U11 pad 11: ISENSE_A -> DUTY
- U11 pad 7: unconnected-(U11-IN3-Pad7) -> VSENSE
- U11 pad 8: unconnected-(U11-IN4-Pad8) -> VSENSE_L
- U11 pad 9: ISENSE_C -> ISENSE
Routing:
- net /10V: track 188.0 -> 473.5 mm, vias 7 -> 10
- net /CTRL_DC: track 0.00 -> 206.6 mm, vias 0 -> 6
- net /Analog_IO/VSENSE_L_IN: track 0.00 -> 201.2 mm, vias 0 -> 10
- net /CTRL_DA: track 0.00 -> 171.6 mm, vias 0 -> 4
- net /CTRL_DB: track 0.00 -> 153.5 mm, vias 0 -> 4
- net /THROTTLE: track 118.5 -> 0.00 mm
- net ISENSE_C_HALL_3: track 0.00 -> 96.7 mm, vias 0 -> 2
- net ISENSE_A_HALL_1: track 0.00 -> 92.9 mm, vias 0 -> 2
- net ISENSE_B_HALL_2: track 0.00 -> 89.7 mm, vias 0 -> 2
- net 5V: track 287.4 -> 364.0 mm, vias 4 -> 5
- net VSENSE: track 103.4 -> 27.6 mm, vias 2 -> 4
- net ISENSE: track 180.1 -> 127.4 mm, vias 7 -> 8
- net /DA_O: track 0.00 -> 51.9 mm
- net THROTTLE: track 0.00 -> 50.5 mm, vias 0 -> 2
- net /DB_O: track 0.00 -> 49.8 mm
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- added copper zone on F.Cu, net LOAD+
Other:
- board outline added: 201.8 x 175 mm
